Commit message: Fix ARES-G headless bring-up: gzserver segfault + kinematics param crash
- Report passive rocker/bogie pivots as state-only joints in ros2_control and
  drop the libgazebo_ros_joint_state_publisher plugin (it threw on load).
- Add enable_cameras xacro arg; wrap the 3 cameras so headless gzserver on
  GPU-less hosts (Codespaces/CI) can skip them and not crash (cameras:=false).
- Lighten LiDAR (24 layers) and remove IMU bias tags for headless stability.
- Fix ares_kinematics_node exit-1: pass publish_tf as a real bool (was a string
  to a bool param). CI ARES smoke test now launches with cameras:=false.

File: rover_ws/src/rover_description/urdf/ares_g.gazebo.xacro (robot description, xacro)
@@ -16,4 +16,7 @@
   <xacro:arg name="controllers_file"
              default="$(find rover_control)/config/ares_controllers.yaml"/>
+  <!-- Camera sensors need a GL/rendering context; disable them for headless
+       gzserver on machines without a GPU (Codespaces) to avoid a crash. -->
+  <xacro:arg name="enable_cameras" default="true"/>
   <!-- ===================== RViz visual materials ===================== -->
   <material name="ares_hull">   <color rgba="0.20 0.22 0.20 1.0"/></material>
@@ -62,19 +65,7 @@
     </plugin>
   </gazebo>
-  <!-- Passive rocker-bogie pivots aren't in ros2_control; publish their state
-       so robot_state_publisher can build the articulated TF tree. -->
-  <gazebo>
-    <plugin name="passive_joint_states" filename="libgazebo_ros_joint_state_publisher.so">
-      <ros>
-        <namespace>/</namespace>
-        <remapping>~/out:=joint_states</remapping>
-      </ros>
-      <update_rate>50</update_rate>
-      <joint_name>left_rocker_joint</joint_name>
-      <joint_name>right_rocker_joint</joint_name>
-      <joint_name>left_bogie_joint</joint_name>
-      <joint_name>right_bogie_joint</joint_name>
-    </plugin>
-  </gazebo>
+  <!-- Passive rocker-bogie pivots are reported as state-only joints inside the
+       ros2_control block, so joint_state_broadcaster publishes them and
+       robot_state_publisher can build the articulated TF tree. -->
   <!-- ===================== LiDAR: Livox Mid-360 class (360 x 59 deg) ===================== -->
   <gazebo reference="lidar_link">
@@ -91,7 +82,8 @@
             <max_angle>3.14159</max_angle>
           </horizontal>
-          <!-- Mid-360 vertical FOV: -7 deg to +52 deg (59 deg total) -->
+          <!-- Mid-360 vertical FOV: -7 deg to +52 deg (59 deg total).
+               24 layers keeps the CPU ray sensor light for headless sim. -->
           <vertical>
-            <samples>40</samples>
+            <samples>24</samples>
             <resolution>1</resolution>
             <min_angle>-0.12217</min_angle>
@@ -128,12 +120,12 @@
       <imu>
         <angular_velocity>
-          <x><noise type="gaussian"><mean>0.0</mean><stddev>1.4e-4</stddev><bias_mean>1e-5</bias_mean><bias_stddev>1e-6</bias_stddev></noise></x>
-          <y><noise type="gaussian"><mean>0.0</mean><stddev>1.4e-4</stddev><bias_mean>1e-5</bias_mean><bias_stddev>1e-6</bias_stddev></noise></y>
-          <z><noise type="gaussian"><mean>0.0</mean><stddev>1.4e-4</stddev><bias_mean>1e-5</bias_mean><bias_stddev>1e-6</bias_stddev></noise></z>
+          <x><noise type="gaussian"><mean>0.0</mean><stddev>1.4e-4</stddev></noise></x>
+          <y><noise type="gaussian"><mean>0.0</mean><stddev>1.4e-4</stddev></noise></y>
+          <z><noise type="gaussian"><mean>0.0</mean><stddev>1.4e-4</stddev></noise></z>
         </angular_velocity>
         <linear_acceleration>
-          <x><noise type="gaussian"><mean>0.0</mean><stddev>1.4e-2</stddev><bias_mean>0.01</bias_mean><bias_stddev>0.001</bias_stddev></noise></x>
-          <y><noise type="gaussian"><mean>0.0</mean><stddev>1.4e-2</stddev><bias_mean>0.01</bias_mean><bias_stddev>0.001</bias_stddev></noise></y>
-          <z><noise type="gaussian"><mean>0.0</mean><stddev>1.4e-2</stddev><bias_mean>0.01</bias_mean><bias_stddev>0.001</bias_stddev></noise></z>
+          <x><noise type="gaussian"><mean>0.0</mean><stddev>1.4e-2</stddev></noise></x>
+          <y><noise type="gaussian"><mean>0.0</mean><stddev>1.4e-2</stddev></noise></y>
+          <z><noise type="gaussian"><mean>0.0</mean><stddev>1.4e-2</stddev></noise></z>
         </linear_acceleration>
       </imu>
@@ -148,4 +140,6 @@
     </sensor>
   </gazebo>
+  <!-- ===================== Cameras (need a GL context; toggle for headless) ===================== -->
+  <xacro:if value="$(arg enable_cameras)">
   <!-- ===================== Forward depth camera: RealSense D455 class ===================== -->
   <gazebo reference="front_cam_link">
@@ -206,3 +200,4 @@
   <xacro:d435i name="left_cam"/>
   <xacro:d435i name="rear_cam"/>
+  </xacro:if>
 </robot>

File: rover_ws/src/rover_description/urdf/ares_g.urdf.xacro (robot description, xacro)
@@ -307,4 +307,13 @@
     </joint>
   </xacro:macro>
+  <!-- Passive (un-actuated) pivots: state-only so joint_state_broadcaster
+       publishes them and robot_state_publisher can build the articulated TF
+       tree (avoids a separate joint_state_publisher plugin). -->
+  <xacro:macro name="passive_ctrl" params="name">
+    <joint name="${name}">
+      <state_interface name="position"/>
+      <state_interface name="velocity"/>
+    </joint>
+  </xacro:macro>
   <ros2_control name="AresGazeboSystem" type="system">
     <hardware>
@@ -321,4 +330,8 @@
     <xacro:steer_ctrl name="left_rear_steer_joint"/>
     <xacro:steer_ctrl name="right_rear_steer_joint"/>
+    <xacro:passive_ctrl name="left_rocker_joint"/>
+    <xacro:passive_ctrl name="right_rocker_joint"/>
+    <xacro:passive_ctrl name="left_bogie_joint"/>
+    <xacro:passive_ctrl name="right_bogie_joint"/>
     <joint name="marker_shoulder_joint">
       <command_interface name="position">

Commit message: Rework ARES-G drive to robust gazebo_ros plugins (drop gazebo_ros2_control)
gazebo_ros2_control on this build forwards the whole URDF to the
controller_manager as a CLI --param and rcl can't parse the XML as YAML, so the
controller_manager never started. Replaced the ros2_control stack with proven
gazebo_ros plugins:
  - libgazebo_ros_diff_drive: six-wheel skid-steer drive + /odom (ARES-G track
    0.28, wheel dia 0.22). Skid-steer is the L0.3 degraded-mode fallback.
  - libgazebo_ros_joint_pose_trajectory: actuates the four real steered kingpins
    and the 2-DOF marker arm.
  - libgazebo_ros_joint_state_publisher: joint states for full articulated TF.
ares_kinematics_node now commands the kingpins via JointTrajectory on
/set_joint_trajectory (Ackermann + skid fallback); marker_arm_node likewise.
Simplified the launch (no controller_manager/spawners/prolog-strip). Updated CI
smoke test + package deps; removed the dead ares_controllers.yaml.

File: rover_ws/src/rover_description/urdf/ares_g.gazebo.xacro (robot description, xacro)
@@ -1,9 +1,9 @@
 <?xml version="1.0"?>
 <!--
-  Gazebo Classic materials, surface physics, ros2_control plugin and the
+  Gazebo Classic materials, surface physics, drive/steering plugins and the
   ARES-G sensor suite (L0.3 6.1). Included from ares_g.urdf.xacro.
-  Actuation is via gazebo_ros2_control (controllers in ares_controllers.yaml);
-  the four-wheel-steering kinematics node (rover_control) maps /cmd_vel onto the
-  wheel-velocity + kingpin-position controllers and publishes /odom.
+  Actuation: gazebo_ros diff-drive for the six wheels (motion + /odom) and the
+  gazebo_ros joint_pose_trajectory plugin for the four steered kingpins + marker
+  arm (commanded by the rover_control steering / marker nodes from /cmd_vel).
   Sensors (as-real-as-sim-allows):
     /points               PointCloud2  Livox Mid-360-class 360 x 59 deg LiDAR
@@ -13,7 +13,7 @@
 -->
 <robot xmlns:xacro="http://www.ros.org/wiki/xacro">
-  <!-- Controller parameter file (also referenced by the ros2_control plugin) -->
-  <xacro:arg name="controllers_file"
-             default="$(find rover_control)/config/ares_controllers.yaml"/>
+  <!-- Motor command topic / odom-TF ownership (mirrors the baseline rover). -->
+  <xacro:arg name="publish_wheel_odom_tf" default="true"/>
+  <xacro:arg name="cmd_vel_topic" default="cmd_vel"/>
   <!-- Camera sensors need a GL/rendering context; disable them for headless
        gzserver on machines without a GPU (Codespaces) to avoid a crash. -->
@@ -57,15 +57,75 @@
   <xacro:wheel_gazebo prefix="rear_left"/>
   <xacro:wheel_gazebo prefix="rear_right"/>
-  <!-- ===================== ros2_control plugin ===================== -->
+  <!-- ===================== Skid-steer drive (3 wheel pairs, ARES-G dims) ===================== -->
+  <!-- Proven gazebo_ros plugin: reliable motion + /odom. Skid-steer is the L0.3
+       degraded-mode fallback; the four kingpins add real steering on top. -->
   <gazebo>
-    <plugin filename="libgazebo_ros2_control.so" name="gazebo_ros2_control">
-      <parameters>$(arg controllers_file)</parameters>
-      <robot_param>robot_description</robot_param>
-      <robot_param_node>robot_state_publisher</robot_param_node>
+    <plugin name="diff_drive" filename="libgazebo_ros_diff_drive.so">
+      <ros>
+        <namespace>/</namespace>
+        <remapping>cmd_vel:=$(arg cmd_vel_topic)</remapping>
+      </ros>
+      <num_wheel_pairs>3</num_wheel_pairs>
+      <left_joint>front_left_wheel_joint</left_joint>
+      <right_joint>front_right_wheel_joint</right_joint>
+      <left_joint>mid_left_wheel_joint</left_joint>
+      <right_joint>mid_right_wheel_joint</right_joint>
+      <left_joint>rear_left_wheel_joint</left_joint>
+      <right_joint>rear_right_wheel_joint</right_joint>
+      <!-- ARES-G: track 0.28 m (centre-centre), wheel dia 0.22 m -->
+      <wheel_separation>0.28</wheel_separation>
+      <wheel_separation>0.28</wheel_separation>
+      <wheel_separation>0.28</wheel_separation>
+      <wheel_diameter>0.22</wheel_diameter>
+      <wheel_diameter>0.22</wheel_diameter>
+      <wheel_diameter>0.22</wheel_diameter>
+      <max_wheel_torque>40.0</max_wheel_torque>
+      <max_wheel_acceleration>2.0</max_wheel_acceleration>
+      <odometry_frame>odom</odometry_frame>
+      <robot_base_frame>base_footprint</robot_base_frame>
+      <publish_odom>true</publish_odom>
+      <publish_odom_tf>$(arg publish_wheel_odom_tf)</publish_odom_tf>
+      <publish_wheel_tf>false</publish_wheel_tf>
+      <update_rate>50.0</update_rate>
     </plugin>
   </gazebo>
-  <!-- Passive rocker-bogie pivots are reported as state-only joints inside the
-       ros2_control block, so joint_state_broadcaster publishes them and
-       robot_state_publisher can build the articulated TF tree. -->
+  <!-- Joint states for ALL joints (wheels, steered kingpins, passive pivots,
+       marker arm) so robot_state_publisher builds the full articulated TF. -->
+  <gazebo>
+    <plugin name="joint_states" filename="libgazebo_ros_joint_state_publisher.so">
+      <ros>
+        <namespace>/</namespace>
+        <remapping>~/out:=joint_states</remapping>
+      </ros>
+      <update_rate>50</update_rate>
+      <joint_name>front_left_wheel_joint</joint_name>
+      <joint_name>front_right_wheel_joint</joint_name>
+      <joint_name>mid_left_wheel_joint</joint_name>
+      <joint_name>mid_right_wheel_joint</joint_name>
+      <joint_name>rear_left_wheel_joint</joint_name>
+      <joint_name>rear_right_wheel_joint</joint_name>
+      <joint_name>left_bogie_steer_joint</joint_name>
+      <joint_name>right_bogie_steer_joint</joint_name>
+      <joint_name>left_rear_steer_joint</joint_name>
+      <joint_name>right_rear_steer_joint</joint_name>
+      <joint_name>left_rocker_joint</joint_name>
+      <joint_name>right_rocker_joint</joint_name>
+      <joint_name>left_bogie_joint</joint_name>
+      <joint_name>right_bogie_joint</joint_name>
+      <joint_name>marker_shoulder_joint</joint_name>
+      <joint_name>marker_elbow_joint</joint_name>
+    </plugin>
+  </gazebo>
+  <!-- Four-station steering + marker arm actuation. The kinematics node
+       publishes a JointTrajectory on /set_joint_trajectory to position the four
+       kingpins (Ackermann angles from /cmd_vel) and the 2-DOF marker arm. -->
+  <gazebo>
+    <plugin name="joint_pose_trajectory" filename="libgazebo_ros_joint_pose_trajectory.so">
+      <ros>
+        <namespace>/</namespace>
+      </ros>
+      <update_rate>50</update_rate>
+    </plugin>
+  </gazebo>
   <!-- ===================== LiDAR: Livox Mid-360 class (360 x 59 deg) ===================== -->
   <gazebo reference="lidar_link">

File: rover_ws/src/rover_description/urdf/ares_g.urdf.xacro (robot description, xacro)
@@ -13,7 +13,7 @@
     * Steering (3.1.2): FOUR STEERED STATIONS as real revolute kingpin joints -
       two rear wheels steer individually, two front bogies steer as rigid units
-      about a shared kingpin. Position-actuated via ros2_control and driven by
-      the four-wheel-steering kinematics node (rover_control), with a skid-steer
-      fallback for in-place turns (as the doc retains).
+      about a shared kingpin. Position-actuated via the joint_pose_trajectory
+      plugin, driven by the four-wheel-steering node (rover_control), with a
+      skid-steer fallback for in-place turns (as the doc retains).
     * Marker arm (6.5): 2-DOF, 0.40 m reach, paint-canister tip.
     * Sensors (6.1): Livox Mid-360-class 360x59 deg LiDAR, forward stereo
@@ -170,6 +170,6 @@
     </joint>
     <!-- STEERED STATION #1/#2: front bogie kingpin (both bogie wheels yaw together).
-         Real revolute kingpin, position-actuated by ros2_control + the
-         four-wheel-steering kinematics node (skid-steer is the fallback mode). -->
+         Real revolute kingpin, position-actuated by the joint_pose_trajectory
+         plugin + the four-wheel-steering node (skid-steer is the fallback). -->
     <joint name="${side}_bogie_steer_joint" type="revolute">
       <parent link="${side}_bogie_carrier"/>
@@ -281,75 +281,12 @@
     <dynamics damping="0.2" friction="0.1"/>
   </joint>
-  <!-- ===================== ros2_control (genuine actuation) ===================== -->
-  <!-- Six drive wheels (velocity) + four steered kingpins (position) + the
-       2-DOF marker arm (position). gazebo_ros2_control loads the controllers
-       named in ares_controllers.yaml. -->
-  <xacro:arg name="controllers_file"
-             default="$(find rover_control)/config/ares_controllers.yaml"/>
-  <xacro:macro name="wheel_ctrl" params="name">
-    <joint name="${name}">
-      <command_interface name="velocity">
-        <param name="min">-20.0</param>
-        <param name="max">20.0</param>
-      </command_interface>
-      <state_interface name="position"/>
-      <state_interface name="velocity"/>
-    </joint>
-  </xacro:macro>
-  <xacro:macro name="steer_ctrl" params="name">
-    <joint name="${name}">
-      <command_interface name="position">
-        <param name="min">${-steer_limit}</param>
-        <param name="max">${steer_limit}</param>
-      </command_interface>
-      <state_interface name="position"/>
-      <state_interface name="velocity"/>
-    </joint>
-  </xacro:macro>
-  <!-- Passive (un-actuated) pivots: state-only so joint_state_broadcaster
-       publishes them and robot_state_publisher can build the articulated TF
-       tree (avoids a separate joint_state_publisher plugin). -->
-  <xacro:macro name="passive_ctrl" params="name">
-    <joint name="${name}">
-      <state_interface name="position"/>
-      <state_interface name="velocity"/>
-    </joint>
-  </xacro:macro>
-  <ros2_control name="AresGazeboSystem" type="system">
-    <hardware>
-      <plugin>gazebo_ros2_control/GazeboSystem</plugin>
-    </hardware>
-    <xacro:wheel_ctrl name="front_left_wheel_joint"/>
-    <xacro:wheel_ctrl name="front_right_wheel_joint"/>
-    <xacro:wheel_ctrl name="mid_left_wheel_joint"/>
-    <xacro:wheel_ctrl name="mid_right_wheel_joint"/>
-    <xacro:wheel_ctrl name="rear_left_wheel_joint"/>
-    <xacro:wheel_ctrl name="rear_right_wheel_joint"/>
-    <xacro:steer_ctrl name="left_bogie_steer_joint"/>
-    <xacro:steer_ctrl name="right_bogie_steer_joint"/>
-    <xacro:steer_ctrl name="left_rear_steer_joint"/>
-    <xacro:steer_ctrl name="right_rear_steer_joint"/>
-    <xacro:passive_ctrl name="left_rocker_joint"/>
-    <xacro:passive_ctrl name="right_rocker_joint"/>
-    <xacro:passive_ctrl name="left_bogie_joint"/>
-    <xacro:passive_ctrl name="right_bogie_joint"/>
-    <joint name="marker_shoulder_joint">
-      <command_interface name="position">
-        <param name="min">${-PI/2}</param>
-        <param name="max">${PI/2}</param>
-      </command_interface>
-      <state_interface name="position"/>
-      <state_interface name="velocity"/>
-    </joint>
-    <joint name="marker_elbow_joint">
-      <command_interface name="position">
-        <param name="min">${-PI/2}</param>
-        <param name="max">${PI/2}</param>
-      </command_interface>
-      <state_interface name="position"/>
-      <state_interface name="velocity"/>
-    </joint>
-  </ros2_control>
-  <!-- Materials + Gazebo plugins -->
+  <!-- ===================== Drive/actuation args ===================== -->
+  <!-- When true, the diff-drive plugin publishes odom->base_footprint (fine for
+       the bare sim); set false when robot_localization owns that TF. -->
+  <xacro:arg name="publish_wheel_odom_tf" default="true"/>
+  <!-- Motor command topic the diff-drive plugin obeys (cmd_vel for the bare sim;
+       /motor/cmd_vel when the safety+HW-bridge stack drives the motors). -->
+  <xacro:arg name="cmd_vel_topic" default="cmd_vel"/>
+  <!-- Materials + Gazebo plugins (drive, steering, sensors) -->
   <xacro:include filename="$(find rover_description)/urdf/ares_g.gazebo.xacro"/>
 </robot>
